File: Hardware/PCB/Eagle Files/DHJSNoiseConsole.brd (EAGLE design)
At the start: 99 x 31 mm, 14 parts

Commit message: PCB Eagle file revision fixes #1, fixes #2, fixes #3, fixes #4
Parts:
- R2: value 2k -> 1k
- VR1, VR2: value 50k -> 100k
Connections:
- net +9V: no longer D1.3
Routing:
- net +9V: track 131.6 -> 123.2 mm
- net N$2: track 33.0 -> 35.1 mm
Changed lines of the file:
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@@
 <?xml version="1.0" encoding="utf-8"?>
 <!DOCTYPE eagle SYSTEM "eagle.dtd">
-<eagle version="7.2.0">
+<eagle version="6.6.0">
 <drawing>
 <settings>
@@
 <layer number="22" name="bPlace" color="7" fill="1" visible="yes" active="yes"/>
 <layer number="23" name="tOrigins" color="15" fill="1" visible="yes" active="yes"/>
-<layer number="24" name="bOrigins" color="15" fill="1" visible="no" active="yes"/>
+<layer number="24" name="bOrigins" color="15" fill="1" visible="yes" active="yes"/>
 <layer number="25" name="tNames" color="7" fill="1" visible="yes" active="yes"/>
-<layer number="26" name="bNames" color="7" fill="1" visible="no" active="yes"/>
+<layer number="26" name="bNames" color="7" fill="1" visible="yes" active="yes"/>
 <layer number="27" name="tValues" color="7" fill="1" visible="yes" active="yes"/>
-<layer number="28" name="bValues" color="7" fill="1" visible="no" active="yes"/>
+<layer number="28" name="bValues" color="7" fill="1" visible="yes" active="yes"/>
 <layer number="29" name="tStop" color="7" fill="3" visible="yes" active="yes"/>
 <layer number="30" name="bStop" color="7" fill="6" visible="yes" active="yes"/>
@@
 <pass name="Default">
 <param name="RoutingGrid" value="50mil"/>
-<param name="AutoGrid" value="1"/>
-<param name="Efforts" value="0"/>
-<param name="TopRouterVariant" value="1"/>
 <param name="tpViaShape" value="round"/>
 <param name="PrefDir.1" value="|"/>
@@
 <attribute name="PROD_#" value="NA" x="95.875" y="15.5" size="1.778" layer="27" rot="R270" display="off"/>
 </element>
-<element name="VR1" library="MusicThingModular" package="9MM_SNAP-IN_POT" value="50k" x="66.04" y="15.5"/>
-<element name="VR2" library="MusicThingModular" package="9MM_SNAP-IN_POT" value="50k" x="16.51" y="15.5"/>
+<element name="VR1" library="MusicThingModular" package="9MM_SNAP-IN_POT" value="100k" x="66.04" y="15.5"/>
+<element name="VR2" library="MusicThingModular" package="9MM_SNAP-IN_POT" value="100k" x="16.51" y="15.5"/>
 <element name="D1" library="SparkFun-LED" package="LED-RGB-THRU" value="LED-RGB-CC-THRUCLEAR" x="41.25" y="14.23" rot="R180">
 <attribute name="PROD_ID" value="DIO-08418" x="41.25" y="14.23" size="1.778" layer="27" rot="R180" display="off"/>
 </element>
 <element name="S2" library="SparkFun-Electromechanical" package="TACTILE-PTH-SIDEEZ" value="" x="80.01" y="2.032"/>
-<element name="R2" library="MusicThingModular" package="10MM_RESISTOR" value="2k" x="30.48" y="7.747"/>
+<element name="R2" library="MusicThingModular" package="10MM_RESISTOR" value="1k" x="30.48" y="7.747"/>
 <element name="U$1" library="TW_logos" package="MTM_1CM_KEEPOUT" value="" x="92.71" y="19.05" rot="MR0"/>
 <element name="U$2" library="MusicThingModular" package="MINI_SPDT_RIGHTANGLE" value="MINI_SPDT" x="80.01" y="28.448" smashed="yes" rot="R270"/>
@@
 <contactref element="NE-556" pad="10"/>
 <contactref element="VR2" pad="3"/>
-<contactref element="D1" pad="3"/>
 <contactref element="S2" pad="1"/>
 <contactref element="U$2" pad="UP"/>
@@
 <wire x1="82.296" y1="28.8036" x2="82.55" y2="28.348" width="0.6096" layer="1"/>
 <wire x1="68.1228" y1="8.6868" x2="68.54" y2="8.5" width="0.6096" layer="1"/>
-<wire x1="42.9768" y1="15.5448" x2="42.0624" y2="14.6304" width="0.6096" layer="1"/>
-<wire x1="49.3776" y1="15.5448" x2="42.9768" y2="15.5448" width="0.6096" layer="1"/>
-<wire x1="42.0624" y1="14.6304" x2="41.885" y2="14.23" width="0.6096" layer="1"/>
-<wire x1="49.3776" y1="15.5448" x2="49.53" y2="15.24" width="0.6096" layer="1"/>
 <wire x1="49.8348" y1="15.0876" x2="50.977440625" y2="13.944959375" width="0.6096" layer="1"/>
 <wire x1="50.977440625" y1="13.944959375" x2="53.73775625" y2="12.8016" width="0.6096" layer="1" curve="45"/>
@@
 <contactref element="S2" pad="2"/>
 <contactref element="U$2" pad="COMMON"/>
-<wire x1="74.5236" y1="9.144" x2="80.735021875" y2="2.932578125" width="0.6096" layer="1"/>
-<wire x1="80.735021875" y1="2.932578125" x2="82.296" y2="2.286" width="0.6096" layer="1" curve="45"/>
-<wire x1="82.296" y1="2.286" x2="82.51" y2="2.032" width="0.6096" layer="1"/>
-<wire x1="74.5236" y1="9.144" x2="74.5236" y2="13.571378125" width="0.6096" layer="1"/>
-<wire x1="74.5236" y1="13.571378125" x2="75.272440625" y2="15.379240625" width="0.6096" layer="1" curve="-44.99995"/>
-<wire x1="75.272440625" y1="15.379240625" x2="77.984" y2="18.0908" width="0.6096" layer="1"/>
-<wire x1="77.984" y1="18.0908" x2="80.01" y2="22.981996875" width="0.6096" layer="1" curve="45"/>
-<wire x1="80.01" y1="22.981996875" x2="80.01" y2="28.548" width="0.6096" layer="1"/>
-<wire x1="74.5236" y1="9.144" x2="73.406" y2="9.144" width="0.6096" layer="1"/>
+<wire x1="82.51" y1="2.032" x2="81.788" y2="2.032" width="0.8128" layer="1"/>
+<wire x1="81.788" y1="2.032" x2="80.75395" y2="3.06605" width="0.8128" layer="1"/>
+<wire x1="80.75395" y1="3.06605" x2="80.01" y2="4.862103125" width="0.8128" layer="1" curve="-45.00007"/>
+<wire x1="80.01" y1="4.862103125" x2="80.01" y2="5.95648125" width="0.8128" layer="1"/>
+<wire x1="80.01" y1="5.95648125" x2="78.833715625" y2="8.796284375" width="0.8128" layer="1" curve="44.999968"/>
+<wire x1="78.833715625" y1="8.796284375" x2="74.40395" y2="13.22605" width="0.8128" layer="1"/>
+<wire x1="74.40395" y1="13.22605" x2="73.66" y2="15.022103125" width="0.8128" layer="1" curve="-45.00007"/>
+<wire x1="73.66" y1="15.022103125" x2="73.66" y2="21.59" width="0.8128" layer="1"/>
+<wire x1="73.66" y1="21.59" x2="73.66" y2="21.844" width="0.8128" layer="1"/>
+<wire x1="73.66" y1="21.844" x2="73.406" y2="22.098" width="0.8128" layer="1"/>
+<wire x1="80.01" y1="28.548" x2="80.01" y2="25.3062875" width="0.8128" layer="1"/>
+<wire x1="80.01" y1="25.3062875" x2="79.178240625" y2="23.298240625" width="0.8128" layer="1" curve="-45"/>
+<wire x1="79.178240625" y1="23.298240625" x2="78.301759375" y2="22.421759375" width="0.8128" layer="1"/>
+<wire x1="78.301759375" y1="22.421759375" x2="76.2937125" y2="21.59" width="0.8128" layer="1" curve="-45"/>
+<wire x1="76.2937125" y1="21.59" x2="73.66" y2="21.59" width="0.8128" layer="1"/>
 </signal>
 <signal name="GND">
@@
 </signal>
 </signals>
+<errors>
+</errors>
 </board>
 </drawing>
