File: Hardware/PCB/Eagle Files/DHJSNoiseConsole.sch (EAGLE design)
At the start: 13 parts

Commit message: PCB Eagle file revision fixes #1, fixes #2, fixes #3, fixes #4
Parts:
- R2: value 2k -> 1k
- VR1, VR2: value 50k -> 100k
Connections:
- net +9V: no longer D1.GREEN_CATHODE
Changed lines of the file:
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@@
 <?xml version="1.0" encoding="utf-8"?>
 <!DOCTYPE eagle SYSTEM "eagle.dtd">
-<eagle version="7.2.0">
+<eagle version="6.6.0">
 <drawing>
 <settings>
@@
 </classes>
 <parts>
-<part name="VR1" library="MusicThingModular" deviceset="9MM_SNAP-IN_POT" device="_" value="50k"/>
-<part name="VR2" library="MusicThingModular" deviceset="9MM_SNAP-IN_POT" device="_" value="50k"/>
+<part name="VR1" library="MusicThingModular" deviceset="9MM_SNAP-IN_POT" device="_" value="100k"/>
+<part name="VR2" library="MusicThingModular" deviceset="9MM_SNAP-IN_POT" device="_" value="100k"/>
 <part name="NE-556" library="SparkFun-AnalogIC" deviceset="556" device=""/>
 <part name="SUPPLY1" library="supply2" deviceset="+9V" device=""/>
@@
 <part name="D1" library="SparkFun-LED" deviceset="LED-RGB-CC-THRU" device="CLEAR"/>
 <part name="SUPPLY11" library="supply2" deviceset="GND" device=""/>
-<part name="SUPPLY12" library="supply2" deviceset="+9V" device=""/>
 <part name="S2" library="SparkFun-Electromechanical" deviceset="SWITCH-MOMENTARY-2" device="SIDE_EZ" value=""/>
-<part name="R2" library="MusicThingModular" deviceset="RESISTOR" device="10MM_RESISTOR" value="2k"/>
+<part name="R2" library="MusicThingModular" deviceset="RESISTOR" device="10MM_RESISTOR" value="1k"/>
 <part name="U$2" library="MusicThingModular" deviceset="MINI_SPDT" device=""/>
 </parts>
@@
 <instance part="D1" gate="G$1" x="76.2" y="15.24"/>
 <instance part="SUPPLY11" gate="GND" x="104.14" y="12.7"/>
-<instance part="SUPPLY12" gate="G$1" x="45.72" y="20.32"/>
 <instance part="S2" gate="G$1" x="-20.32" y="76.2" rot="R270"/>
 <instance part="R2" gate="G$1" x="93.98" y="15.24" rot="R180"/>
@@
 <wire x1="73.66" y1="96.52" x2="73.66" y2="93.98" width="0.1524" layer="91"/>
 </segment>
-<segment>
-<pinref part="SUPPLY12" gate="G$1" pin="+9V"/>
-<wire x1="45.72" y1="15.24" x2="45.72" y2="17.78" width="0.1524" layer="91"/>
-<pinref part="D1" gate="G$1" pin="GREEN_CATHODE"/>
-<wire x1="43.18" y1="15.24" x2="45.72" y2="15.24" width="0.1524" layer="91"/>
-<label x="43.18" y="15.24" size="1.778" layer="95" rot="R180" xref="yes"/>
-<junction x="45.72" y="15.24"/>
-<wire x1="45.72" y1="15.24" x2="71.12" y2="15.24" width="0.1524" layer="91"/>
-</segment>
 </net>
